File: Hardware/Electronics/CAD/Remote.kicad_sch (KiCad schematic)
At the start: 49 parts, among them J1 CONN_01X01, J2 CONN_01X01, J3 CONN_02X03, J4 CONN_01X06, J5 CONN_01X12, J6 CONN_01X24, Q1 SI1308EDL, Q2 BC817, Q3 BC817, U1 ATmega328P-A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

Commit message: fix expander in schematics and pcb design
Connections:
- net +3V3: now also U3.18 (~{RESET})
- net Earth: now also U3.15 (A0), U3.16 (A1), U3.17 (A2); no longer U3.18 (~{RESET})
- no-connect marks 21 -> 18
Changed lines of the file:
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@@
   (junction (at 250.19 80.01) (diameter 0) (color 0 0 0 0)
   )
+  (junction (at 173.99 157.48) (diameter 0) (color 0 0 0 0)
+  )
   (junction (at 52.07 90.17) (diameter 0) (color 0 0 0 0)
   )
   (junction (at 260.35 114.3) (diameter 0) (color 0 0 0 0)
   )
+  (junction (at 153.67 148.59) (diameter 0) (color 0 0 0 0)
+  )
   (junction (at 260.35 137.16) (diameter 0) (color 0 0 0 0)
   )
@@
   (junction (at 198.12 122.555) (diameter 0) (color 0 0 0 0)
   )
+  (junction (at 153.67 146.05) (diameter 0) (color 0 0 0 0)
+  )
   (junction (at 118.11 41.91) (diameter 0) (color 0 0 0 0)
   )
   (junction (at 250.19 120.65) (diameter 0) (color 0 0 0 0)
   )
-  (junction (at 199.39 130.81) (diameter 0) (color 0 0 0 0)
-  )
   (junction (at 198.12 110.49) (diameter 0) (color 0 0 0 0)
   )
@@
   (no_connect (at 191.77 148.59))
   (no_connect (at 57.15 66.04))
-  (no_connect (at 156.21 148.59))
   (no_connect (at 64.77 135.89))
   (no_connect (at 34.29 105.41))
@@
   (no_connect (at 267.97 26.67))
   (no_connect (at 64.77 133.35))
-  (no_connect (at 156.21 146.05))
   (no_connect (at 64.77 105.41))
   (no_connect (at 191.77 125.73))
@@
   (no_connect (at 64.77 156.21))
   (no_connect (at 64.77 130.81))
-  (no_connect (at 156.21 143.51))
   (no_connect (at 191.77 123.19))
   (no_connect (at 34.29 107.95))
@@
     (stroke (width 0) (type default))
   )
+  (wire (pts (xy 153.67 143.51) (xy 153.67 146.05))
+    (stroke (width 0) (type default))
+  )
   (wire (pts (xy 242.57 58.42) (xy 242.57 57.15))
     (stroke (width 0) (type default))
@@
     (stroke (width 0) (type default))
   )
-  (wire (pts (xy 199.39 130.81) (xy 199.39 131.445))
-    (stroke (width 0) (type default))
-  )
   (wire (pts (xy 64.77 125.73) (xy 69.85 125.73))
     (stroke (width 0) (type default))
@@
     (stroke (width 0) (type default))
   )
-  (wire (pts (xy 200.66 130.81) (xy 199.39 130.81))
-    (stroke (width 0) (type default))
-  )
   (wire (pts (xy 267.97 44.45) (xy 264.16 44.45))
     (stroke (width 0) (type default))
@@
     (stroke (width 0) (type default))
   )
-  (wire (pts (xy 173.99 156.21) (xy 173.99 158.75))
+  (wire (pts (xy 173.99 156.21) (xy 173.99 157.48))
     (stroke (width 0) (type default))
   )
@@
     (stroke (width 0) (type default))
   )
+  (wire (pts (xy 173.99 157.48) (xy 173.99 158.75))
+    (stroke (width 0) (type default))
+  )
   (wire (pts (xy 76.2 110.49) (xy 76.2 101.6))
     (stroke (width 0) (type default))
@@
     (stroke (width 0) (type default))
   )
-  (wire (pts (xy 199.39 130.81) (xy 191.77 130.81))
+  (wire (pts (xy 191.77 130.81) (xy 200.66 130.81))
     (stroke (width 0) (type default))
   )
@@
     (stroke (width 0) (type default))
   )
+  (wire (pts (xy 153.67 148.59) (xy 153.67 157.48))
+    (stroke (width 0) (type default))
+  )
   (wire (pts (xy 161.925 62.23) (xy 158.75 62.23))
     (stroke (width 0) (type default))
@@
     (stroke (width 0) (type default))
   )
+  (wire (pts (xy 153.67 146.05) (xy 153.67 148.59))
+    (stroke (width 0) (type default))
+  )
   (wire (pts (xy 48.26 64.77) (xy 50.8 64.77))
     (stroke (width 0) (type default))
@@
     (stroke (width 0) (type default))
   )
+  (wire (pts (xy 153.67 157.48) (xy 173.99 157.48))
+    (stroke (width 0) (type default))
+  )
   (wire (pts (xy 64.77 107.95) (xy 73.66 107.95))
     (stroke (width 0) (type default))
@@
     (stroke (width 0) (type default))
   )
+  (wire (pts (xy 156.21 143.51) (xy 153.67 143.51))
+    (stroke (width 0) (type default))
+  )
   (wire (pts (xy 195.58 140.97) (xy 191.77 140.97))
     (stroke (width 0) (type default))
@@
     (stroke (width 0) (type default))
   )
+  (wire (pts (xy 153.67 146.05) (xy 156.21 146.05))
+    (stroke (width 0) (type default))
+  )
   (wire (pts (xy 247.65 137.16) (xy 250.19 137.16))
     (stroke (width 0) (type default))
@@
     (stroke (width 0) (type default))
   )
+  (wire (pts (xy 153.67 148.59) (xy 156.21 148.59))
+    (stroke (width 0) (type default))
+  )
   (wire (pts (xy 191.77 138.43) (xy 196.85 138.43))
     (stroke (width 0) (type default))
@@
     )
   )
-  (symbol (lib_id "Remote-rescue:Earth") (at 153.67 130.81 270) (mirror x) (unit 1)
-    (in_bom yes) (on_board yes) (dnp no)
-    (property "Reference" "#PWR029" (at 147.32 130.81 0)
-      (effects (font (size 1.27 1.27)) hide)
-    )
-    (property "Value" "Earth" (at 149.86 130.81 0)
-      (effects (font (size 1.27 1.27)) hide)
-    )
-    (property "Footprint" "" (at 153.67 130.81 0)
-      (effects (font (size 1.27 1.27)) hide)
-    )
-    (property "Datasheet" "" (at 153.67 130.81 0)
-      (effects (font (size 1.27 1.27)) hide)
-    )
-    (pin "1")
-    (instances
-      (project "Remote"
-        (path "/68f488c0-7fea-4096-b751-b5ed1b6acab1"
-          (reference "#PWR029") (unit 1)
-        )
-      )
-    )
-  )
   (symbol (lib_id "Remote-rescue:R") (at 204.47 114.3 90) (mirror x) (unit 1)
     (in_bom yes) (on_board yes) (dnp no)
@@
         )
       )
+    )
+  )
+  (symbol (lib_id "Remote-rescue:+3V3") (at 153.67 130.81 90) (mirror x) (unit 1)
+    (in_bom yes) (on_board yes) (dnp no)
+    (property "Reference" "#PWR029" (at 157.48 130.81 0)
+      (effects (font (size 1.27 1.27)) hide)
+    )
+    (property "Value" "+3V3" (at 147.955 130.81 90)
+      (effects (font (size 1.27 1.27)))
+    )
+    (property "Footprint" "" (at 153.67 130.81 0)
+      (effects (font (size 1.27 1.27)) hide)
+    )
+    (property "Datasheet" "" (at 153.67 130.81 0)
+      (effects (font (size 1.27 1.27)) hide)
+    )
+    (pin "1")
+    (instances
+      (project "Remote"
+        (path "/68f488c0-7fea-4096-b751-b5ed1b6acab1"
+          (reference "#PWR029") (unit 1)
+        )
+      )

Commit message: Change IR led resistor from 330 to 33 Ohm
Parts:
- R2: value 330 -> 33
Changed lines of the file:
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@@
       (effects (font (size 1.27 1.27)))
     )
-    (property "Value" "330" (at 142.24 173.99 90)
+    (property "Value" "33" (at 142.24 173.99 90)
       (effects (font (size 1.27 1.27)))
     )
